File: schematics/uvfoto-avr.sch (EAGLE design)
At the start: 3 parts, among them IC1 MEGA128-A, IC2 L298

Commit message: Updated schematics
Parts:
- added IC3: LMV324M, linear:LMV324M
- added R1, R4: 20K, rcl:R-EU_0207/10
- added R2, R3: 2M, rcl:R-EU_0207/10
Connections:
- net N$1 renamed HOME_POS_SW
- new net BLDC_A: IC3A.+IN
- new net BLDC_B: IC3B.+IN
- new net IO_PHASE_1: IC3A.OUT, R2.2
- new net N$6: IC3A.-IN, R1.2, R2.1
- new net N$8: IC3B.-IN, R3.1, R4.2
- new net N$9: IC3B.OUT, R3.2
- net GND: now also IC3P.V-, R1.1, R4.1
- net VCC: now also IC3P.V+
Changed lines of the file:
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@@
 <layer number="97" name="Info" color="7" fill="1" visible="yes" active="yes"/>
 <layer number="98" name="Guide" color="6" fill="1" visible="yes" active="yes"/>
+<layer number="99" name="SpiceOrder" color="5" fill="1" visible="yes" active="yes"/>
 </layers>
 <schematic xreflabel="%F%N/%S.%C%R" xrefpart="/%S.%C%R">
@@
 <part name="P+1" library="supply1" deviceset="VCC" device=""/>
 <part name="P+2" library="supply1" deviceset="VCC" device=""/>
+<part name="IC3" library="linear" deviceset="LMV324?*" device="M"/>
+<part name="P+3" library="supply1" deviceset="VCC" device=""/>
+<part name="GND3" library="supply1" deviceset="GND" device=""/>
+<part name="R2" library="rcl" deviceset="R-EU_" device="0207/10" value="2M"/>
+<part name="R1" library="rcl" deviceset="R-EU_" device="0207/10" value="20K"/>
+<part name="GND4" library="supply1" deviceset="GND" device=""/>
+<part name="R3" library="rcl" deviceset="R-EU_" device="0207/10" value="2M"/>
+<part name="R4" library="rcl" deviceset="R-EU_" device="0207/10" value="20K"/>
+<part name="GND5" library="supply1" deviceset="GND" device=""/>
 </parts>
 <sheets>
@@
 <instance part="P+1" gate="VCC" x="96.52" y="83.82"/>
 <instance part="P+2" gate="VCC" x="81.28" y="83.82"/>
+<instance part="IC3" gate="A" x="182.88" y="38.1"/>
+<instance part="IC3" gate="P" x="182.88" y="38.1"/>
+<instance part="IC3" gate="B" x="182.88" y="7.62"/>
+<instance part="IC3" gate="C" x="185.42" y="-12.7"/>
+<instance part="IC3" gate="D" x="185.42" y="-33.02"/>
+<instance part="P+3" gate="VCC" x="182.88" y="48.26"/>
+<instance part="GND3" gate="1" x="182.88" y="27.94"/>
+<instance part="R2" gate="G$1" x="182.88" y="20.32"/>
+<instance part="R1" gate="G$1" x="157.48" y="35.56"/>
+<instance part="GND4" gate="1" x="152.4" y="25.4"/>
+<instance part="R3" gate="G$1" x="180.34" y="-2.54"/>
+<instance part="R4" gate="G$1" x="157.48" y="5.08"/>
+<instance part="GND5" gate="1" x="152.4" y="-5.08"/>
 </instances>
 <busses>
@@
 <wire x1="104.14" y1="53.34" x2="99.06" y2="53.34" width="0.1524" layer="91"/>
 </segment>
-</net>
-<net name="N$1" class="0">
+<segment>
+<pinref part="IC3" gate="P" pin="V-"/>
+<pinref part="GND3" gate="1" pin="GND"/>
+</segment>
+<segment>
+<pinref part="R1" gate="G$1" pin="1"/>
+<pinref part="GND4" gate="1" pin="GND"/>
+<wire x1="152.4" y1="35.56" x2="152.4" y2="27.94" width="0.1524" layer="91"/>
+</segment>
+<segment>
+<pinref part="R4" gate="G$1" pin="1"/>
+<pinref part="GND5" gate="1" pin="GND"/>
+<wire x1="152.4" y1="5.08" x2="152.4" y2="-2.54" width="0.1524" layer="91"/>
+</segment>
+</net>
+<net name="HOME_POS_SW" class="0">
 <segment>
 <pinref part="IC1" gate="G$1" pin="(SCL/INT0)PD0"/>
 <wire x1="66.04" y1="5.08" x2="93.98" y2="5.08" width="0.1524" layer="91"/>
 <pinref part="S1" gate="1" pin="S"/>
+<label x="73.66" y="5.08" size="1.778" layer="95"/>
 </segment>
 </net>
@@
 <wire x1="104.14" y1="76.2" x2="104.14" y2="71.12" width="0.1524" layer="91"/>
 </segment>
+<segment>
+<pinref part="IC3" gate="P" pin="V+"/>
+<pinref part="P+3" gate="VCC" pin="VCC"/>
+</segment>
 </net>
 <net name="UART_TX" class="0">
@@
 </segment>
 </net>
+<net name="BLDC_A" class="0">
+<segment>
+<pinref part="IC3" gate="A" pin="+IN"/>
+<wire x1="175.26" y1="40.64" x2="165.1" y2="40.64" width="0.1524" layer="91"/>
+<label x="162.56" y="40.64" size="1.778" layer="95"/>
+</segment>
+</net>
+<net name="IO_PHASE_1" class="0">
+<segment>
+<pinref part="IC3" gate="A" pin="OUT"/>
+<wire x1="190.5" y1="38.1" x2="198.12" y2="38.1" width="0.1524" layer="91"/>
+<pinref part="R2" gate="G$1" pin="2"/>
+<wire x1="198.12" y1="38.1" x2="200.66" y2="38.1" width="0.1524" layer="91"/>
+<wire x1="187.96" y1="20.32" x2="198.12" y2="20.32" width="0.1524" layer="91"/>
+<wire x1="198.12" y1="20.32" x2="198.12" y2="38.1" width="0.1524" layer="91"/>
+</segment>
+</net>
+<net name="N$6" class="0">
+<segment>
+<pinref part="R2" gate="G$1" pin="1"/>
+<wire x1="177.8" y1="20.32" x2="167.64" y2="20.32" width="0.1524" layer="91"/>
+<wire x1="167.64" y1="20.32" x2="167.64" y2="35.56" width="0.1524" layer="91"/>
+<wire x1="162.56" y1="35.56" x2="167.64" y2="35.56" width="0.1524" layer="91"/>
+<pinref part="IC3" gate="A" pin="-IN"/>
+<wire x1="167.64" y1="35.56" x2="175.26" y2="35.56" width="0.1524" layer="91"/>
+<pinref part="R1" gate="G$1" pin="2"/>
+</segment>
+</net>
+<net name="BLDC_B" class="0">
+<segment>
+<pinref part="IC3" gate="B" pin="+IN"/>
+<wire x1="165.1" y1="10.16" x2="175.26" y2="10.16" width="0.1524" layer="91"/>
+<label x="162.56" y="10.16" size="1.778" layer="95"/>
+</segment>
+</net>
+<net name="N$8" class="0">
+<segment>
+<pinref part="IC3" gate="B" pin="-IN"/>
+<wire x1="175.26" y1="5.08" x2="170.18" y2="5.08" width="0.1524" layer="91"/>
+<pinref part="R3" gate="G$1" pin="1"/>
+<wire x1="170.18" y1="5.08" x2="162.56" y2="5.08" width="0.1524" layer="91"/>
+<wire x1="175.26" y1="-2.54" x2="170.18" y2="-2.54" width="0.1524" layer="91"/>
+<wire x1="170.18" y1="-2.54" x2="170.18" y2="5.08" width="0.1524" layer="91"/>
+<pinref part="R4" gate="G$1" pin="2"/>
+</segment>
+</net>
+<net name="N$9" class="0">
+<segment>
+<pinref part="IC3" gate="B" pin="OUT"/>
+<wire x1="190.5" y1="7.62" x2="200.66" y2="7.62" width="0.1524" layer="91"/>
+<wire x1="200.66" y1="7.62" x2="200.66" y2="-2.54" width="0.1524" layer="91"/>
+<pinref part="R3" gate="G$1" pin="2"/>
+<wire x1="200.66" y1="-2.54" x2="185.42" y2="-2.54" width="0.1524" layer="91"/>
+</segment>
+</net>
