File: schematics/kicad/laser_peripherals.sch (KiCad schematic (older format))
At the start: 15 parts, among them Q1 BC547, Q2 BC547, U1 LM358, U2 LM339

Commit message: Updated schematics
Parts:
- added SW1: SW_PUSH, ~, symbol SW_PUSH
Connections:
- net GND: now also SW1.1
- net MCU/STEP_HOME_POS: now also SW1.2
- net TEST: now reaches R2.2, U1.1
- net DIODE_OUT renamed LED_DETECTOR_OUT
- net LASER_DRIVER_PULSE renamed laser_driver.sch/LASER_PULSE
- net LASER_DRIVER_PWM renamed laser_driver.sch/LASER_PWM
Changed lines of the file:
@@
-EESchema Schematic File Version 2  date Tue 30 Apr 2013 06:08:21 PM EEST
-LIBS:stellaris_launchpad
+EESchema Schematic File Version 2  date otrdiena, 2013. gada 30. aprīlis, plkst. 20 un 12
 LIBS:power
 LIBS:device
@@
 LIBS:contrib
 LIBS:valves
-LIBS:noname-cache
+LIBS:laser_peripherals-cache
 EELAYER 27 0
 EELAYER END
 $Descr A4 11693 8268
 encoding utf-8
-Sheet 1 2
+Sheet 1 4
 Title ""
 Date "30 apr 2013"
@@
 	5050 2150 5050 1400
 Wire Wire Line
-	5950 1300 5750 1300
+	5750 1300 6000 1300
 Wire Wire Line
 	5900 1300 5900 700
@@
 Connection ~ 2300 3700
 Wire Wire Line
-	2650 3400 3050 3400
+	2650 3400 4900 3400
 Connection ~ 2650 3400
-Text GLabel 3050 3400 2    60   Input ~ 0
-LASER_DRIVER_PULSE
 Text GLabel 1600 3700 0    60   Input ~ 0
 LASER_PULSE_MCU
@@
 Connection ~ 2300 5350
 Wire Wire Line
-	2650 5050 3050 5050
+	2650 5050 5550 5050
 Connection ~ 2650 5050
-Text GLabel 3050 5050 2    60   Input ~ 0
-LASER_DRIVER_PWM
 Text GLabel 1600 5350 0    60   Input ~ 0
 LASER_PWM_MCU
@@
 Text GLabel 9400 2800 0    60   Input ~ 0
 LASER_PULSE_MCU
+$Comp
+L SW_PUSH SW1
+U 1 1 517FEECC
+P 8400 3700
+F 0 "SW1" H 8550 3810 50  0000 C CNN
+F 1 "SW_PUSH" H 8400 3620 50  0000 C CNN
+F 2 "~" H 8400 3700 60  0000 C CNN
+F 3 "~" H 8400 3700 60  0000 C CNN
+	1    8400 3700
+	1    0    0    -1
+$EndComp
+$Comp
+L GND #PWR011
+U 1 1 517FEEDB
+P 7950 3850
+F 0 "#PWR011" H 7950 3850 30  0001 C CNN
+F 1 "GND" H 7950 3780 30  0001 C CNN
+F 2 "" H 7950 3850 60  0000 C CNN
+F 3 "" H 7950 3850 60  0000 C CNN
+	1    7950 3850
+	1    0    0    -1
+$EndComp
+Wire Wire Line
+	8700 3700 9400 3700
+Wire Wire Line
+	8100 3700 7950 3700
+Wire Wire Line
+	7950 3700 7950 3850
+Text Label 4000 1550 0    60   ~ 0
+TEST
+Text Label 5950 1300 0    60   ~ 0
+OUTPUT
+Text Label 6000 1300 0    60   ~ 0
+LABEL
+Text GLabel 5950 1300 2    60   Input ~ 0
+LED_DETECTOR_OUT
+Text GLabel 9400 2650 0    60   Output ~ 0
+LED_DETECTOR_OUT
+$Sheet
+S 9250 5050 1450 1650
+U 51800D74
+F0 "Power" 50
+F1 "power.sch" 50
+$EndSheet
+$Sheet
+S 5700 4200 1100 1650
+U 518010D7
+F0 "laser_driver.sch" 50
+F1 "laser_driver.sch" 50
+F2 "LASER_PWM" I L 5700 4350 60
+F3 "LASER_PULSE" I L 5700 4500 60
+$EndSheet
+Wire Wire Line
+	4900 3400 4900 4500
+Wire Wire Line
+	4900 4500 5700 4500
+Wire Wire Line
+	5550 5050 5550 4350
+Wire Wire Line
+	5550 4350 5700 4350
 $EndSCHEMATC

Commit message: Updated schematics
Parts:
- removed D1: LED, ~, symbol LED
- removed Q1, Q2: BC547, TO92, symbol BC547
- removed R1: 5K, ~, symbol R
- removed R10, R5, R6, R7, R8, R9: 900R, ~, symbol R
- removed R2: R, ~, symbol R
- removed R3, R4: 10K, ~, symbol R
- removed U1: LM358, symbol LM358
- removed U2: LM339, symbol LM339
- added U1: L298_BREAKOUT, ~, symbol L298_BREAKOUT
Connections:
- net GND: now also U1.11 (GND)
- net MCU/STEP_A1: now also U1.1 (INPUT1)
- net MCU/STEP_A2: now also U1.2 (INPUT2)
- net MCU/STEP_B1: now also U1.3 (INPUT3)
- net MCU/STEP_B2: now also U1.4 (INPUT4)
- net VCC: now also U1.5 (EN)
- new net +12V: U1.10 (VDD)
- no-connect marks 0 -> 2
Other:
- note added: "Motor EN and CLK go to laser printer head motor\n"
