File: schematics/kicad/mcu.sch (KiCad schematic (older format))
At the start: 1 part, among them U4 STELLARIS_LAUNCHPAD

Commit message: Updated schematics
Connections:
- no-connect marks 0 -> 29
Changed lines of the file:
@@
-EESchema Schematic File Version 2  date Tue 30 Apr 2013 06:08:21 PM EEST
-LIBS:stellaris_launchpad
+EESchema Schematic File Version 2  date otrdiena, 2013. gada 30. aprīlis, plkst. 20 un 12
 LIBS:power
 LIBS:device
@@
 LIBS:contrib
 LIBS:valves
-LIBS:noname-cache
+LIBS:laser_peripherals-cache
 EELAYER 27 0
 EELAYER END
 $Descr A4 11693 8268
 encoding utf-8
-Sheet 2 2
+Sheet 2 4
 Title ""
 Date "30 apr 2013"
@@
 	2600 2650 2600 2750
 $Comp
-L GND #PWR011
+L GND #PWR012
 U 1 1 517FDBED
 P 2600 2750
-F 0 "#PWR011" H 2600 2750 30  0001 C CNN
+F 0 "#PWR012" H 2600 2750 30  0001 C CNN
 F 1 "GND" H 2600 2680 30  0001 C CNN
 F 2 "" H 2600 2750 60  0000 C CNN
@@
 Text HLabel 3750 3150 0    60   Input ~ 0
 STEP_HOME_POS
+NoConn ~ 3750 2350
+NoConn ~ 3750 2450
+NoConn ~ 3750 3350
+NoConn ~ 3750 3550
+NoConn ~ 3750 3650
+NoConn ~ 3750 3850
+NoConn ~ 3750 3950
+NoConn ~ 3750 4050
+NoConn ~ 3750 4150
+NoConn ~ 3750 4250
+NoConn ~ 5550 4250
+NoConn ~ 5550 4150
+NoConn ~ 5550 4050
+NoConn ~ 5550 3950
+NoConn ~ 5550 3850
+NoConn ~ 5550 3750
+NoConn ~ 5550 3550
+NoConn ~ 5550 3450
+NoConn ~ 5550 3350
+NoConn ~ 5550 3250
+NoConn ~ 5550 3150
+NoConn ~ 5550 3050
+NoConn ~ 5550 2950
+NoConn ~ 5550 2850
+NoConn ~ 5550 2750
+NoConn ~ 5550 2650
+NoConn ~ 5550 2550
+NoConn ~ 5550 2450
+NoConn ~ 5550 2350
 $EndSCHEMATC

Commit message: Updated schematics
Connections:
- net VCC: now reaches U4.2 (VBUS)
- no-connect marks 29 -> 28
Changed lines of the file:
@@
-EESchema Schematic File Version 2  date otrdiena, 2013. gada 30. aprīlis, plkst. 20 un 12
+EESchema Schematic File Version 2  date trešdiena, 2013. gada  1. maijs, plkst. 00 un 49
 LIBS:power
 LIBS:device
@@
 LIBS:contrib
 LIBS:valves
+LIBS:l298_breakout
+LIBS:stellaris_launchpad
 LIBS:laser_peripherals-cache
 EELAYER 27 0
@@
 encoding utf-8
 Sheet 2 4
-Title ""
+Title "Lasershow"
 Date "30 apr 2013"
 Rev ""
-Comp ""
+Comp "Hackerspace"
 Comment1 ""
 Comment2 ""
@@
 	2600 2650 2600 2750
 $Comp
-L GND #PWR012
+L GND #PWR05
 U 1 1 517FDBED
 P 2600 2750
-F 0 "#PWR012" H 2600 2750 30  0001 C CNN
+F 0 "#PWR05" H 2600 2750 30  0001 C CNN
 F 1 "GND" H 2600 2680 30  0001 C CNN
 F 2 "" H 2600 2750 60  0000 C CNN
@@
 STEP_HOME_POS
 NoConn ~ 3750 2350
-NoConn ~ 3750 2450
 NoConn ~ 3750 3350
 NoConn ~ 3750 3550
@@
 NoConn ~ 5550 2450
 NoConn ~ 5550 2350
+$Comp
+L VCC #PWR06
+U 1 1 51802907
+P 3250 2300
+F 0 "#PWR06" H 3250 2400 30  0001 C CNN
+F 1 "VCC" H 3250 2400 30  0000 C CNN
+F 2 "" H 3250 2300 60  0000 C CNN
+F 3 "" H 3250 2300 60  0000 C CNN
+	1    3250 2300
+	1    0    0    -1
+$EndComp
+Wire Wire Line
+	3250 2300 3250 2450
+Wire Wire Line
+	3250 2450 3750 2450
 $EndSCHEMATC
