File: schematics/kicad/power.sch (KiCad schematic (older format))
At the start: 4 parts, among them CON1 BARREL_JACK, U3 7805

Commit message: Updated schematics
Changed lines of the file:
@@
-EESchema Schematic File Version 2  date otrdiena, 2013. gada 30. aprīlis, plkst. 20 un 12
+EESchema Schematic File Version 2  date trešdiena, 2013. gada  1. maijs, plkst. 00 un 49
 LIBS:power
 LIBS:device
@@
 LIBS:contrib
 LIBS:valves
+LIBS:l298_breakout
+LIBS:stellaris_launchpad
 LIBS:laser_peripherals-cache
 EELAYER 27 0
@@
 encoding utf-8
 Sheet 3 4
-Title ""
+Title "Lasershow"
 Date "30 apr 2013"
 Rev ""
-Comp ""
+Comp "Hackerspace"
 Comment1 ""
 Comment2 ""
@@
 	3100 1900 3100 2250
 $Comp
-L GND #PWR013
+L GND #PWR07
 U 1 1 51800DB8
 P 3100 2250
-F 0 "#PWR013" H 3100 2250 30  0001 C CNN
+F 0 "#PWR07" H 3100 2250 30  0001 C CNN
 F 1 "GND" H 3100 2180 30  0001 C CNN
 F 2 "" H 3100 2250 60  0000 C CNN
@@
 $EndComp
 $Comp
-L GND #PWR014
+L GND #PWR08
 U 1 1 51800DC7
 P 4200 2150
-F 0 "#PWR014" H 4200 2150 30  0001 C CNN
+F 0 "#PWR08" H 4200 2150 30  0001 C CNN
 F 1 "GND" H 4200 2080 30  0001 C CNN
 F 2 "" H 4200 2150 60  0000 C CNN
@@
 Connection ~ 4750 1700
 $Comp
-L VCC #PWR015
+L VCC #PWR09
 U 1 1 51800E14
 P 5100 1700
-F 0 "#PWR015" H 5100 1800 30  0001 C CNN
+F 0 "#PWR09" H 5100 1800 30  0001 C CNN
 F 1 "VCC" H 5100 1800 30  0000 C CNN
 F 2 "" H 5100 1700 60  0000 C CNN
@@
 $EndComp
 $Comp
-L +12V #PWR016
+L +12V #PWR010
 U 1 1 51800F13
 P 3250 1600
-F 0 "#PWR016" H 3250 1550 20  0001 C CNN
+F 0 "#PWR010" H 3250 1550 20  0001 C CNN
 F 1 "+12V" H 3250 1700 30  0000 C CNN
 F 2 "" H 3250 1600 60  0000 C CNN
@@
 Wire Wire Line
 	3250 1600 3250 1700
+$Comp
+L PWR_FLAG #FLG011
+U 1 1 51805F5F
+P 2900 1700
+F 0 "#FLG011" H 2900 1795 30  0001 C CNN
+F 1 "PWR_FLAG" H 2900 1880 30  0000 C CNN
+F 2 "" H 2900 1700 60  0000 C CNN
+F 3 "" H 2900 1700 60  0000 C CNN
+	1    2900 1700
+	1    0    0    -1
+$EndComp
 $EndSCHEMATC
