File: schematics/kicad/laser_driver.sch (KiCad schematic (older format))
At the start: 28 parts, among them Q3 BC547, Q4 BC547, Q5 BD237, Q6 MOSFET_N, U2 LM358, U5 LM339

Commit message: Updated schematics to match the code (and, reality)
Parts:
- added R5: 100R, ~, symbol R
Connections:
- net GND: now also R5.2
Changed lines of the file:
@@
-EESchema Schematic File Version 2  date ceturtdiena, 2013. gada  9. maijs, plkst. 01 un 37
+EESchema Schematic File Version 2  date svētdiena, 2013. gada 19. maijs, plkst. 23 un 38
 LIBS:power
 LIBS:device
@@
 Sheet 4 4
 Title "Lasershow"
-Date "8 may 2013"
+Date "19 may 2013"
 Rev ""
 Comp "Hackerspace"
@@
 $EndComp
 $Comp
-L VCC #PWR012
+L VCC #PWR20
 U 1 1 51801199
 P 8300 3600
-F 0 "#PWR012" H 8300 3700 30  0001 C CNN
+F 0 "#PWR20" H 8300 3700 30  0001 C CNN
 F 1 "VCC" H 8300 3700 30  0000 C CNN
 F 2 "" H 8300 3600 60  0000 C CNN
@@
 	8300 4250 8300 4400
 $Comp
-L +12V #PWR013
+L +12V #PWR21
 U 1 1 518011E0
 P 9950 3600
-F 0 "#PWR013" H 9950 3550 20  0001 C CNN
+F 0 "#PWR21" H 9950 3550 20  0001 C CNN
 F 1 "+12V" H 9950 3700 30  0000 C CNN
 F 2 "" H 9950 3600 60  0000 C CNN
@@
 $EndComp
 $Comp
-L GND #PWR014
+L GND #PWR22
 U 1 1 518012C9
 P 9950 6950
-F 0 "#PWR014" H 9950 6950 30  0001 C CNN
+F 0 "#PWR22" H 9950 6950 30  0001 C CNN
 F 1 "GND" H 9950 6880 30  0001 C CNN
 F 2 "" H 9950 6950 60  0000 C CNN
@@
 $EndComp
 $Comp
-L GND #PWR015
+L GND #PWR19
 U 1 1 518012D8
 P 7550 6150
-F 0 "#PWR015" H 7550 6150 30  0001 C CNN
+F 0 "#PWR19" H 7550 6150 30  0001 C CNN
 F 1 "GND" H 7550 6080 30  0001 C CNN
 F 2 "" H 7550 6150 60  0000 C CNN
@@
 $EndComp
 $Comp
-L GND #PWR016
+L GND #PWR14
 U 1 1 5180284D
 P 3150 7150
-F 0 "#PWR016" H 3150 7150 30  0001 C CNN
+F 0 "#PWR14" H 3150 7150 30  0001 C CNN
 F 1 "GND" H 3150 7080 30  0001 C CNN
 F 2 "" H 3150 7150 60  0000 C CNN
@@
 	2250 6850 2100 6850
 $Comp
-L VCC #PWR017
+L VCC #PWR13
 U 1 1 51802856
 P 3150 5850
-F 0 "#PWR017" H 3150 5950 30  0001 C CNN
+F 0 "#PWR13" H 3150 5950 30  0001 C CNN
 F 1 "VCC" H 3150 5950 30  0000 C CNN
 F 2 "" H 3150 5850 60  0000 C CNN
@@
 $EndComp
 $Comp
-L GND #PWR018
+L GND #PWR18
 U 1 1 5180492C
 P 5000 1850
-F 0 "#PWR018" H 5000 1850 30  0001 C CNN
+F 0 "#PWR18" H 5000 1850 30  0001 C CNN
 F 1 "GND" H 5000 1780 30  0001 C CNN
 F 2 "" H 5000 1850 60  0000 C CNN
@@
 $EndComp
 $Comp
-L VCC #PWR019
+L VCC #PWR17
 U 1 1 51804932
 P 5000 1250
-F 0 "#PWR019" H 5000 1350 30  0001 C CNN
+F 0 "#PWR17" H 5000 1350 30  0001 C CNN
 F 1 "VCC" H 5000 1350 30  0000 C CNN
 F 2 "" H 5000 1250 60  0000 C CNN
@@
 $EndComp
 $Comp
-L VCC #PWR020
+L VCC #PWR15
 U 1 1 51804938
 P 4200 1850
-F 0 "#PWR020" H 4200 1950 30  0001 C CNN
+F 0 "#PWR15" H 4200 1950 30  0001 C CNN
 F 1 "VCC" H 4200 1950 30  0000 C CNN
 F 2 "" H 4200 1850 60  0000 C CNN
@@
 $EndComp
 $Comp
-L GND #PWR021
+L GND #PWR16
 U 1 1 5180493E
 P 4200 2950
-F 0 "#PWR021" H 4200 2950 30  0001 C CNN
+F 0 "#PWR16" H 4200 2950 30  0001 C CNN
 F 1 "GND" H 4200 2880 30  0001 C CNN
 F 2 "" H 4200 2950 60  0000 C CNN
@@
 $EndComp
 $Comp
-L VCC #PWR022
+L VCC #PWR11
 U 1 1 5180495C
 P 2700 1300
-F 0 "#PWR022" H 2700 1400 30  0001 C CNN
+F 0 "#PWR11" H 2700 1400 30  0001 C CNN
 F 1 "VCC" H 2700 1400 30  0000 C CNN
 F 2 "" H 2700 1300 60  0000 C CNN
@@
 $EndComp
 $Comp
-L GND #PWR023
+L GND #PWR12
 U 1 1 51804962
 P 2700 2300
-F 0 "#PWR023" H 2700 2300 30  0001 C CNN
+F 0 "#PWR12" H 2700 2300 30  0001 C CNN
 F 1 "GND" H 2700 2230 30  0001 C CNN
 F 2 "" H 2700 2300 60  0000 C CNN
@@
 Text Notes 3650 2550 2    60   ~ 0
 Start of line detector- reverse biased blue LED,\n amplified and fed to schmitt trigger\n
+$Comp
+L R R5
+U 1 1 51993818
+P 10200 5600
+F 0 "R5" V 10280 5600 40  0000 C CNN
+F 1 "100R" V 10207 5601 40  0000 C CNN
+F 2 "~" V 10130 5600 30  0000 C CNN
+F 3 "~" H 10200 5600 30  0000 C CNN
+	1    10200 5600
+	0    -1   -1   0
+$EndComp
+$Comp
+L GND #PWR23
+U 1 1 5199382C
+P 10450 5800
+F 0 "#PWR23" H 10450 5800 30  0001 C CNN
+F 1 "GND" H 10450 5730 30  0001 C CNN
+F 2 "" H 10450 5800 60  0000 C CNN
+F 3 "" H 10450 5800 60  0000 C CNN
+	1    10450 5800
+	1    0    0    -1
+$EndComp
+Wire Wire Line
+	10450 5600 10450 5800
 $EndSCHEMATC

Commit message: Moving on with line drawing algorithms
Parts:
- R14: value 1K5 -> 390R
Changed lines of the file:
@@
-EESchema Schematic File Version 2  date svētdiena, 2013. gada 19. maijs, plkst. 23 un 38
+EESchema Schematic File Version 2  date trešdiena, 2013. gada 22. maijs, plkst. 20 un 28
 LIBS:power
 LIBS:device
@@
 Sheet 4 4
 Title "Lasershow"
-Date "19 may 2013"
+Date "22 may 2013"
 Rev ""
 Comp "Hackerspace"
@@
 P 7050 4050
 F 0 "R14" V 7130 4050 40  0000 C CNN
-F 1 "1K5" V 7057 4051 40  0000 C CNN
+F 1 "390R" V 7057 4051 40  0000 C CNN
 F 2 "~" V 6980 4050 30  0000 C CNN
 F 3 "~" H 7050 4050 30  0000 C CNN
